File: hardware/wiegand-bridge.kicad_pcb (KiCad board)
At the start: 4 copper layers, 90 x 95 mm, 195 parts, among them J1 USB-C, J10 READER D0 D1, J11 READER LED BEEP, J12 GND IN3, J13 IN4 GND, J14 DC IN, J15 RELAY NC NO, J16 RELAY COM, J17 W5500, J18 QWIIC, J19 EXPANSION, J2 6-36V IN, J20 RS485 A B, J21 RS485 12V GND, J3 READER PWR, J4 LiFePO4 + NTC, J5 OLED SOCKET, J6 TFT/EPD, J8 TAMPER EXT, J9 IN1 IN2, K1 SRD-05VDC-SL-C, Q1 2N7002, Q10 2N7002, Q11 AO3401A, Q12 AO3400A, Q2 2N7002, Q4 2N7002, Q5 AO3401A, Q6 FS8205A, Q7 2N7002, Q8 2N7002, Q9 2N7002, SW1 BOOT, SW2 RESET, SW3 TAMPER, U1 ESP32-S3-WROOM-1-N8R2, U10 LMV321, U2 LMR16020, U3 TPS63001, U4 SN74LVC2G17, U5 CN3058E, U6 MT3608, U7 DW01A, U8 TCA9535, U9 SP3485

Commit message: rev 10b: back silkscreen links wiegand.edgecoil.dev
Silkscreen-only change (the CERN-OHL-S source location). Copper, mask, paste, drill, outline, BOM
and CPL are unchanged; DRC results are identical to rev 10.
Other:
- board text added: "rev 10b 2026-10"
- board text added: "wiegand.edgecoil.dev"
- board text removed: "edgecoil.dev"
- board text removed: "rev 10 2026-10"
Changed lines of the file:
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@@
 		)
 	)
-	(gr_text "edgecoil.dev"
+	(gr_text "wiegand.edgecoil.dev"
 		(at 158 164.277087 0)
 		(layer "B.SilkS")
@@
 		)
 	)
-	(gr_text "rev 10  2026-10"
+	(gr_text "rev 10b  2026-10"
 		(at 158 162.077087 0)
 		(layer "B.SilkS")
