File: hardware/lite/wiegand-bridge-lite.kicad_pcb (KiCad board)
At the start: 4 copper layers, 42 x 44 mm, 75 parts, among them J1 USB-C, J3 12V GND D0 D1 LED BEEP A B, Q1 2N7002, Q2 2N7002, Q3 2N7002, Q4 2N7002, SW1 BOOT, SW2 RESET, U1 ESP32-S3-MINI-1-N4R2, U11 SN74LVC2G17, U2 AP63203, U4 SN74LVC2G17, U9 SP3485

Commit message: LITE: TVS swapped to the Preferred SMAJ18A (no loading fee, 54k stock); re-routed, fab outputs and renders regenerated; cost note
Parts:
- D2: footprint SMA_L4.4-W2.6-LS5.0-R-RD -> SMA_L4.3-W2.6-LS5.0-RD
Connections:
- D2 pad 1: GND -> +VIN
- D2 pad 2: +VIN -> GND
Routing:
- net +3V3: track 164.1 -> 147.7 mm, vias 3 -> 6
- net D0_TX: track 24.1 -> 37.8 mm, vias 3 -> 2
- net D0_RAW: track 23.7 -> 33.9 mm, vias 0 -> 1
- net D1_TX: track 29.0 -> 19.1 mm, vias 2 -> 3
- net +VIN: track 67.4 -> 58.4 mm, vias 3 -> 2
- net RDR_LED: track 22.6 -> 29.6 mm
- net RS485_B: track 26.5 -> 32.5 mm, vias 1 -> 0
- net RDR_BEEP: track 30.7 -> 26.3 mm, vias 1 -> 0
- net WG_D0: track 21.3 -> 17.8 mm
- net USB_DP: track 10.9 -> 14.3 mm
- net IO21: track 23.2 -> 19.8 mm
- net IO47: track 22.0 -> 18.9 mm
- net +VIN_F: track 9.38 -> 12.1 mm
- net LED_TX: track 14.5 -> 16.8 mm, vias 2 -> 3
- net BEEP_RX: track 12.3 -> 14.7 mm
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